File: LibMake.sch (KiCad schematic (older format))
At the start: 22 parts

Commit message: Uodate L.lib
Parts:
- removed L?: L, ~, symbol L
- removed LED?: LED, ~, symbol LED
- removed R?: R-TYPE1, ~, symbol R-TYPE1
- added L?: L-TYPE1, ~, symbol L-TYPE1
- added L?: L-TYPE2, ~, symbol L-TYPE2
- added L?: L-TYPE3, ~, symbol L-TYPE3
- added LED?: LED, ~, symbol LED
- added R?: R-TYPE1, ~, symbol R-TYPE1
Other:
- moved on the sheet: D?
