File: LibMake.sch (KiCad schematic (older format))
At the start: 24 parts

Commit message: Update
Parts:
- removed Q?: FET-N, ~, symbol FET-N
- removed Q?: FET-P, ~, symbol FET-P
- removed Q?: TR-NPN, ~, symbol TR-NPN
- removed Q?: TR-PNP, ~, symbol TR-PNP
- removed Q?: JFET-N, ~, symbol JFET-N
- removed Q?: JFET-P, ~, symbol JFET-P
- added Q?: TR-NPN, ~, symbol TR-NPN
- added Q?: TR-PNP, ~, symbol TR-PNP
- added Q?: JFET-P, ~, symbol JFET-P
- added Q?: JFET-N, ~, symbol JFET-N
- added Q?: FET-N, ~, symbol FET-N
- added Q?: FET-P, ~, symbol FET-P
- added SW?: SW-SPST, ~, symbol SW-SPST
- added SW?: SW-SPDT, ~, symbol SW-SPDT
- added SW?: SW-DPST, ~, symbol SW-DPST
- added SW?: SW-DPST-TACT, ~, symbol SW-DPST-TACT
- added SW?: SW-SPST-TACT, ~, symbol SW-SPST-TACT
- added SW?: SW-DPST-TACT-2, ~, symbol SW-DPST-TACT-2
Other:
- moved on the sheet: D?, LED?

Commit message: Update
Parts:
- removed CN?: CON-MALE-01, ~, symbol CON-MALE-01
- removed CN?: CON-MALE-02, ~, symbol CON-MALE-02
- removed CN?: CON-MALE-03, ~, symbol CON-MALE-03
- removed CN?: CON-MALE-04, ~, symbol CON-MALE-04
- removed CN?: CON-MALE-05, ~, symbol CON-MALE-05
- removed CN?: CON-MALE-06, ~, symbol CON-MALE-06
- added CN?: CON-MALE-SINGLE-001, ~, symbol CON-MALE-SINGLE-001
- added CN?: CON-MALE-SINGLE-002, ~, symbol CON-MALE-SINGLE-002
- added CN?: CON-MALE-SINGLE-003, ~, symbol CON-MALE-SINGLE-003
- added CN?: CON-FEMALE-SINGLE-001, ~, symbol CON-FEMALE-SINGLE-001
- added CN?: CON-FEMALE-SINGLE-002, ~, symbol CON-FEMALE-SINGLE-002
- added CN?: CON-FEMALE-SINGLE-003, ~, symbol CON-FEMALE-SINGLE-003
Changed lines of the file:
@@
-EESchema Schematic File Version 2  date 2013/03/30 2:36:10
+EESchema Schematic File Version 2  date 2013/03/30 3:13:40
 LIBS:C
 LIBS:D
@@
 $EndComp
 $Comp
-L CON-MALE-01 CN?
-U 1 1 51538410
-P 6450 4850
-F 0 "CN?" H 6400 4930 40  0000 L CNN
-F 1 "CON-MALE-01" H 6450 4760 40  0000 C CNN
-F 2 "~" H 6400 4850 60  0000 C CNN
-F 3 "~" H 6400 4850 60  0000 C CNN
-	1    6450 4850
-	1    0    0    -1
-$EndComp
-$Comp
-L CON-MALE-02 CN?
-U 1 1 5153841F
-P 6450 4550
-F 0 "CN?" H 6400 4680 40  0000 L CNN
-F 1 "CON-MALE-02" H 6450 4410 40  0000 C CNN
-F 2 "~" H 6400 4600 60  0000 C CNN
-F 3 "~" H 6400 4600 60  0000 C CNN
-	1    6450 4550
-	1    0    0    -1
-$EndComp
-$Comp
-L CON-MALE-03 CN?
-U 1 1 5153842E
-P 6450 4150
-F 0 "CN?" H 6400 4330 40  0000 L CNN
-F 1 "CON-MALE-03" H 6450 3960 40  0000 C CNN
-F 2 "~" H 6400 4250 60  0000 C CNN
-F 3 "~" H 6400 4250 60  0000 C CNN
-	1    6450 4150
-	1    0    0    -1
-$EndComp
-$Comp
-L CON-MALE-04 CN?
-U 1 1 5153843D
-P 6450 3650
-F 0 "CN?" H 6400 3880 40  0000 L CNN
-F 1 "CON-MALE-04" H 6450 3410 40  0000 C CNN
-F 2 "~" H 6400 3800 60  0000 C CNN
-F 3 "~" H 6400 3800 60  0000 C CNN
-	1    6450 3650
-	1    0    0    -1
-$EndComp
-$Comp
-L CON-MALE-05 CN?
-U 1 1 5153844C
-P 6950 4650
-F 0 "CN?" H 6900 4930 40  0000 L CNN
-F 1 "CON-MALE-05" H 6950 4360 40  0000 C CNN
-F 2 "~" H 6900 4850 60  0000 C CNN
-F 3 "~" H 6900 4850 60  0000 C CNN
-	1    6950 4650
-	1    0    0    -1
-$EndComp
-$Comp
-L CON-MALE-06 CN?
-U 1 1 5153845B
-P 6950 3950
-F 0 "CN?" H 6900 4280 40  0000 L CNN
-F 1 "CON-MALE-06" H 6950 3610 40  0000 C CNN
-F 2 "~" H 6900 4200 60  0000 C CNN
-F 3 "~" H 6900 4200 60  0000 C CNN
-	1    6950 3950
-	1    0    0    -1
-$EndComp
-$Comp
 L L-TYPE1 L?
 U 1 1 5155168E
@@
 	1    0    0    -1
 $EndComp
+$Comp
+L CON-MALE-SINGLE-001 CN?
+U 1 1 5155DBCE
+P 6600 4850
+F 0 "CN?" H 6550 4930 40  0000 L CNN
+F 1 "CON-MALE-SINGLE-001" H 6650 4760 40  0000 C CNN
+F 2 "~" H 6550 4850 60  0000 C CNN
+F 3 "~" H 6550 4850 60  0000 C CNN
+	1    6600 4850
+	1    0    0    -1
+$EndComp
+$Comp
+L CON-MALE-SINGLE-002 CN?
+U 1 1 5155DBDD
+P 6600 4550
+F 0 "CN?" H 6550 4680 40  0000 L CNN
+F 1 "CON-MALE-SINGLE-002" H 6650 4410 40  0000 C CNN
+F 2 "~" H 6550 4600 60  0000 C CNN
+F 3 "~" H 6550 4600 60  0000 C CNN
+	1    6600 4550
+	1    0    0    -1
+$EndComp
+$Comp
+L CON-MALE-SINGLE-003 CN?
+U 1 1 5155DBEC
+P 6600 4150
+F 0 "CN?" H 6550 4330 40  0000 L CNN
+F 1 "CON-MALE-SINGLE-003" H 6650 3960 40  0000 C CNN
+F 2 "~" H 6550 4250 60  0000 C CNN
+F 3 "~" H 6550 4250 60  0000 C CNN
+	1    6600 4150
+	1    0    0    -1
+$EndComp
+$Comp
+L CON-FEMALE-SINGLE-001 CN?
+U 1 1 5155DBFB
+P 7450 4850
+F 0 "CN?" H 7400 4930 40  0000 L CNN
+F 1 "CON-FEMALE-SINGLE-001" H 7500 4760 40  0000 C CNN
+F 2 "~" H 7400 4850 60  0000 C CNN
+F 3 "~" H 7400 4850 60  0000 C CNN
+	1    7450 4850
+	1    0    0    -1
+$EndComp
+$Comp
+L CON-FEMALE-SINGLE-002 CN?
+U 1 1 5155DC14
+P 7450 4550
+F 0 "CN?" H 7400 4680 40  0000 L CNN
+F 1 "CON-FEMALE-SINGLE-002" H 7500 4410 40  0000 C CNN
+F 2 "~" H 7400 4600 60  0000 C CNN
+F 3 "~" H 7400 4600 60  0000 C CNN
+	1    7450 4550
+	1    0    0    -1
+$EndComp
+$Comp
+L CON-FEMALE-SINGLE-003 CN?
+U 1 1 5155DC23
+P 7450 4150
+F 0 "CN?" H 7400 4330 40  0000 L CNN
+F 1 "CON-FEMALE-SINGLE-003" H 7500 3960 40  0000 C CNN
+F 2 "~" H 7400 4250 60  0000 C CNN
+F 3 "~" H 7400 4250 60  0000 C CNN
+	1    7450 4150
+	1    0    0    -1
+$EndComp

Commit message: Update
Connector generator is finished.
Parts:
- added CN?: CON-MALE-DOUBLE-098, ~, symbol CON-MALE-DOUBLE-098
- added CN?: CON-FEMALE-DOUBLE-008, ~, symbol CON-FEMALE-DOUBLE-008
- added CN?: CON-MALE-DOUBLE-006, ~, symbol CON-MALE-DOUBLE-006
Changed lines of the file:
@@
-EESchema Schematic File Version 2  date 2013/03/30 3:13:40
+EESchema Schematic File Version 2  date 2013/03/30 4:39:45
 LIBS:C
 LIBS:D
@@
 	1    0    0    -1
 $EndComp
+$Comp
+L CON-MALE-DOUBLE-098 CN?
+U 1 1 5155EB06
+P 8700 4250
+F 0 "CN?" H 8550 6730 40  0000 L CNN
+F 1 "CON-MALE-DOUBLE-098" H 8700 1760 40  0000 C CNN
+F 2 "~" H 8650 6675 60  0000 C CNN
+F 3 "~" H 8650 6675 60  0000 C CNN
+	1    8700 4250
+	1    0    0    -1
+$EndComp
+$Comp
+L CON-FEMALE-DOUBLE-008 CN?
+U 1 1 5155EEE5
+P 7600 5400
+F 0 "CN?" H 7450 5630 40  0000 L CNN
+F 1 "CON-FEMALE-DOUBLE-008" H 7600 5160 40  0000 C CNN
+F 2 "~" H 7550 5575 60  0000 C CNN
+F 3 "~" H 7550 5575 60  0000 C CNN
+	1    7600 5400
+	1    0    0    -1
+$EndComp
+$Comp
+L CON-MALE-DOUBLE-006 CN?
+U 1 1 5155EEF4
+P 6800 5350
+F 0 "CN?" H 6650 5530 40  0000 L CNN
+F 1 "CON-MALE-DOUBLE-006" H 6800 5160 40  0000 C CNN
+F 2 "~" H 6750 5475 60  0000 C CNN
+F 3 "~" H 6750 5475 60  0000 C CNN
+	1    6800 5350
+	1    0    0    -1
+$EndComp

Commit message: Update
Add supply lib
Parts:
- removed CN?: CON-MALE-DOUBLE-098, ~, symbol CON-MALE-DOUBLE-098
- added U1, U2: 74HC04, ~, symbol 74HC04
- added U3, U4: 74HC02, ~, symbol 74HC02
- gave numbers to parts that had none: 32
Connections:
- net labels added: +10V, -5V

Commit message: Update
Parts:
- removed U1, U2: 74HC04, ~, symbol 74HC04
- removed U3, U4: 74HC02, ~, symbol 74HC02
Connections:
- net labels added: +11.1V, -10V
- net labels removed: +10V, -5V
Changed lines of the file:
@@
-EESchema Schematic File Version 2  date 2013/03/31 8:58:28
+EESchema Schematic File Version 2  date 2013/03/31 11:18:13
 LIBS:C
 LIBS:D
@@
 LIBS:SW
 LIBS:Tr
-LIBS:powersupply
 LIBS:connector-female
 LIBS:connector-male
+LIBS:supply1
+LIBS:supply2
 LIBS:device
 LIBS:74xx
@@
 Sheet 1 1
 Title ""
-Date "30 mar 2013"
+Date "31 mar 2013"
 Rev ""
 Comp ""
@@
 $EndComp
 $Comp
-L 74HC04 U1
-U 3 1 51571173
-P 7100 2150
-F 0 "U1" H 7250 2250 40  0000 C CNN
-F 1 "74HC04" H 7300 2050 40  0000 C CNN
-F 2 "~" H 7100 2150 60  0000 C CNN
-F 3 "~" H 7100 2150 60  0000 C CNN
-	3    7100 2150
-	1    0    0    -1
-$EndComp
-$Comp
-L 74HC04 U1
-U 4 1 51571182
-P 7100 2550
-F 0 "U1" H 7250 2650 40  0000 C CNN
-F 1 "74HC04" H 7300 2450 40  0000 C CNN
-F 2 "~" H 7100 2550 60  0000 C CNN
-F 3 "~" H 7100 2550 60  0000 C CNN
-	4    7100 2550
-	1    0    0    -1
-$EndComp
-$Comp
-L 74HC04 U1
-U 5 1 51571191
-P 7100 2950
-F 0 "U1" H 7250 3050 40  0000 C CNN
-F 1 "74HC04" H 7300 2850 40  0000 C CNN
-F 2 "~" H 7100 2950 60  0000 C CNN
-F 3 "~" H 7100 2950 60  0000 C CNN
-	5    7100 2950
-	1    0    0    -1
-$EndComp
-$Comp
-L 74HC04 U1
-U 6 1 51571A10
-P 7100 3300
-F 0 "U1" H 7250 3400 40  0000 C CNN
-F 1 "74HC04" H 7300 3200 40  0000 C CNN
-F 2 "~" H 7100 3300 60  0000 C CNN
-F 3 "~" H 7100 3300 60  0000 C CNN
-	6    7100 3300
-	1    0    0    -1
-$EndComp
-$Comp
-L 74HC04 U2
-U 1 1 51571A1F
-P 7100 3650
-F 0 "U2" H 7250 3750 40  0000 C CNN
-F 1 "74HC04" H 7300 3550 40  0000 C CNN
-F 2 "~" H 7100 3650 60  0000 C CNN
-F 3 "~" H 7100 3650 60  0000 C CNN
-	1    7100 3650
-	1    0    0    -1
-$EndComp
-$Comp
-L 74HC04 U1
-U 1 1 51571A2E
-P 7100 1450
-F 0 "U1" H 7250 1550 40  0000 C CNN
-F 1 "74HC04" H 7300 1350 40  0000 C CNN
-F 2 "~" H 7100 1450 60  0000 C CNN
-F 3 "~" H 7100 1450 60  0000 C CNN
-	1    7100 1450
-	1    0    0    -1
-$EndComp
-$Comp
-L 74HC04 U1
-U 2 1 51571A3D
-P 7100 1800
-F 0 "U1" H 7250 1900 40  0000 C CNN
-F 1 "74HC04" H 7300 1700 40  0000 C CNN
-F 2 "~" H 7100 1800 60  0000 C CNN
-F 3 "~" H 7100 1800 60  0000 C CNN
-	2    7100 1800
-	1    0    0    -1
-$EndComp
-$Comp
-L 74HC02 U3
-U 1 1 51572573
-P 8400 1550
-F 0 "U3" H 8400 1600 60  0000 C CNN
-F 1 "74HC02" H 8450 1500 60  0000 C CNN
-F 2 "~" H 8400 1550 60  0000 C CNN
-F 3 "~" H 8400 1550 60  0000 C CNN
-	1    8400 1550
-	1    0    0    -1
-$EndComp
-$Comp
-L 74HC02 U3
-U 2 1 51572582
-P 8400 2000
-F 0 "U3" H 8400 2050 60  0000 C CNN
-F 1 "74HC02" H 8450 1950 60  0000 C CNN
-F 2 "~" H 8400 2000 60  0000 C CNN
-F 3 "~" H 8400 2000 60  0000 C CNN
-	2    8400 2000
-	1    0    0    -1
-$EndComp
-$Comp
-L 74HC02 U3
-U 3 1 51572591
-P 8400 2450
-F 0 "U3" H 8400 2500 60  0000 C CNN
-F 1 "74HC02" H 8450 2400 60  0000 C CNN
-F 2 "~" H 8400 2450 60  0000 C CNN
-F 3 "~" H 8400 2450 60  0000 C CNN
-	3    8400 2450
-	1    0    0    -1
-$EndComp
-$Comp
-L 74HC02 U3
-U 4 1 515725A0
-P 8400 2900
-F 0 "U3" H 8400 2950 60  0000 C CNN
-F 1 "74HC02" H 8450 2850 60  0000 C CNN
-F 2 "~" H 8400 2900 60  0000 C CNN
-F 3 "~" H 8400 2900 60  0000 C CNN
-	4    8400 2900
-	1    0    0    -1
-$EndComp
-$Comp
-L 74HC02 U4
-U 1 1 515725AF
-P 8400 3350
-F 0 "U4" H 8400 3400 60  0000 C CNN
-F 1 "74HC02" H 8450 3300 60  0000 C CNN
-F 2 "~" H 8400 3350 60  0000 C CNN
-F 3 "~" H 8400 3350 60  0000 C CNN
-	1    8400 3350
-	1    0    0    -1
-$EndComp
-$Comp
-L +10V #PWR?
-U 1 1 51577C74
-P 6100 3550
-F 0 "#PWR?" H 6100 3730 40  0001 C CNN
-F 1 "+10V" H 6100 3675 40  0000 C CNN
-F 2 "~" H 6100 3550 60  0000 C CNN
-F 3 "~" H 6100 3550 60  0000 C CNN
-	1    6100 3550
-	1    0    0    -1
-$EndComp
-$Comp
-L -5V #PWR?
-U 1 1 51577D86
-P 6400 3300
-F 0 "#PWR?" H 6400 3105 40  0001 C CNN
-F 1 "-5V" H 6400 3160 40  0000 C CNN
-F 2 "~" H 6400 3300 -60 0000 C CNN
-F 3 "~" H 6400 3300 -60 0000 C CNN
-	1    6400 3300
-	1    0    0    -1
-$EndComp
+L +11.1V #PWR?
+U 1 1 5157A02F
+P 6300 3200
+F 0 "#PWR?" H 6300 3380 40  0001 C CNN
+F 1 "+11.1V" H 6300 3325 40  0000 C CNN
+F 2 "~" H 6300 3200 60  0000 C CNN
+F 3 "~" H 6300 3200 60  0000 C CNN
+	1    6300 3200
+	1    0    0    -1
+$EndComp
+$Comp
+L -10V #PWR?
+U 1 1 5157A064
+P 6300 3300
+F 0 "#PWR?" H 6300 3105 40  0001 C CNN
+F 1 "-10V" H 6300 3160 40  0000 C CNN
+F 2 "~" H 6300 3300 60  0000 C CNN
+F 3 "~" H 6300 3300 60  0000 C CNN
+	1    6300 3300
+	1    0    0    -1
+$EndComp

Commit message: Update supply lib
Connections:
- net labels added: GND2
Changed lines of the file:
@@
-EESchema Schematic File Version 2  date 2013/03/31 11:18:13
+EESchema Schematic File Version 2  date 2013/03/31 12:12:59
 LIBS:C
 LIBS:D
@@
 LIBS:connector-female
 LIBS:connector-male
+LIBS:supply2
 LIBS:supply1
-LIBS:supply2
 LIBS:device
 LIBS:74xx
+LIBS:power
 LIBS:LibMake-cache
 EELAYER 27 0
@@
 	1    0    0    -1
 $EndComp
+$Comp
+L GND2 #PWR?
+U 1 1 5157A7C4
+P 6500 3300
+F 0 "#PWR?" H 6500 3105 40  0001 C CNN
+F 1 "GND2" H 6500 3160 40  0000 C CNN
+F 2 "~" H 6500 3300 60  0000 C CNN
+F 3 "~" H 6500 3300 60  0000 C CNN
+	1    6500 3300
+	1    0    0    -1
+$EndComp
