File: LibMake.sch (KiCad schematic (older format))
At the start: 32 parts, among them CN1 CON-MALE-SINGLE-003, CN2 CON-MALE-SINGLE-002, CN3 CON-MALE-SINGLE-001, CN4 CON-MALE-DOUBLE-006, CN5 CON-FEMALE-SINGLE-003, CN6 CON-FEMALE-SINGLE-002, CN7 CON-FEMALE-SINGLE-001, CN8 CON-FEMALE-DOUBLE-008, Q1 TR-NPN, Q2 JFET-P, Q3 FET-N, Q4 TR-PNP, Q5 JFET-N, Q6 FET-P, SW1 SW-DPST-TACT-2, SW2 SW-DPST-TACT, SW3 SW-SPST-TACT, SW4 SW-DPST, SW5 SW-SPST, SW6 SW-SPDT

Commit message: Update
Parts:
- removed C1: C-TYPE3, ~, symbol C-TYPE3
- removed C2: C-TYPE2, ~, symbol C-TYPE2
- removed C3: C-TYPE1, ~, symbol C-TYPE1
- removed CN1: CON-MALE-SINGLE-003, ~, symbol CON-MALE-SINGLE-003
- removed CN2: CON-MALE-SINGLE-002, ~, symbol CON-MALE-SINGLE-002
- removed CN3: CON-MALE-SINGLE-001, ~, symbol CON-MALE-SINGLE-001
- removed CN4: CON-MALE-DOUBLE-006, ~, symbol CON-MALE-DOUBLE-006
- removed CN5: CON-FEMALE-SINGLE-003, ~, symbol CON-FEMALE-SINGLE-003
- removed CN6: CON-FEMALE-SINGLE-002, ~, symbol CON-FEMALE-SINGLE-002
- removed CN7: CON-FEMALE-SINGLE-001, ~, symbol CON-FEMALE-SINGLE-001
- removed CN8: CON-FEMALE-DOUBLE-008, ~, symbol CON-FEMALE-DOUBLE-008
- removed LED1: LED, ~, symbol LED
- removed R1: R-TYPE2, ~, symbol R-TYPE2
- removed R2: R-TYPE1, ~, symbol R-TYPE1
- added C?: C(CERA), ~, symbol C(CERA)
- added C?: C(POLE), ~, symbol C(POLE)
- added C?: C(NPOLE), ~, symbol C(NPOLE)
- added CN?: CON-FEMALE-DOUBLE-10, ~, symbol CON-FEMALE-DOUBLE-10
- added CN?: CON-MALE-DOUBLE-10, ~, symbol CON-MALE-DOUBLE-10
- added LED?: LED(PHI5), ~, symbol LED(PHI5)
- added R?: R(1005M), ~, symbol R(1005M)
Changed lines of the file:
@@
-EESchema Schematic File Version 2  date 2013/04/04 23:13:54
-LIBS:C
-LIBS:D
-LIBS:FET
-LIBS:JFET
-LIBS:L
-LIBS:LED
-LIBS:R
-LIBS:SW
-LIBS:Tr
-LIBS:supply2
-LIBS:supply1
+EESchema Schematic File Version 2  date 2013/04/11 11:13:55
+LIBS:Capacitor
+LIBS:ConFe
+LIBS:ConMa
+LIBS:MOSFET
+LIBS:PowerSupply
+LIBS:Resistor
+LIBS:Transistor
+LIBS:PhotoDevice
+LIBS:74xx
 LIBS:device
-LIBS:74xx
-LIBS:power
 LIBS:LibMake-cache
 EELAYER 27 0
@@
 Sheet 1 1
 Title ""
-Date "31 mar 2013"
+Date "11 apr 2013"
 Rev ""
 Comp ""
@@
 $EndComp
 $Comp
-L R-TYPE2 R1
-U 1 1 51520442
-P 5050 4400
-F 0 "R1" H 4925 4460 40  0000 L CNN
-F 1 "R-TYPE2" H 5050 4330 40  0000 C CNN
-F 2 "~" V 4980 4400 30  0000 C CNN
-F 3 "~" H 5050 4400 30  0000 C CNN
-F 4 "4.7k" H 5075 4460 35  0000 L CNN "抵抗値"
-	1    5050 4400
-	1    0    0    -1
-$EndComp
-$Comp
 L DSCH D2
 U 1 1 5151FC8B
@@
 $EndComp
 $Comp
-L C-TYPE1 C3
-U 1 1 5153050F
-P 4950 4850
-F 0 "C3" H 4960 4920 40  0000 L CNN
-F 1 "C-TYPE1" H 4960 4775 40  0000 L CNN
-F 2 "~" H 4988 4700 30  0000 C CNN
-F 3 "~" H 4950 4850 60  0000 C CNN
-F 4 "4.7p" H 5025 4850 35  0000 L CNN "静電容量"
-	1    4950 4850
-	1    0    0    -1
-$EndComp
-$Comp
-L C-TYPE2 C2
-U 1 1 51530528
-P 4650 4850
-F 0 "C2" H 4660 4920 40  0000 L CNN
-F 1 "C-TYPE2" H 4660 4775 40  0000 L CNN
-F 2 "~" H 4688 4700 30  0000 C CNN
-F 3 "~" H 4650 4850 60  0000 C CNN
-F 4 "4.7p" H 4725 4850 35  0000 L CNN "静電容量"
-	1    4650 4850
-	1    0    0    -1
-$EndComp
-$Comp
-L C-TYPE3 C1
-U 1 1 51530541
-P 4350 4850
-F 0 "C1" H 4360 4920 40  0000 L CNN
-F 1 "C-TYPE3" H 4360 4775 40  0000 L CNN
-F 2 "~" H 4388 4700 30  0000 C CNN
-F 3 "~" H 4350 4850 60  0000 C CNN
-F 4 "4.7p" H 4425 4850 35  0000 L CNN "静電容量"
-	1    4350 4850
-	1    0    0    -1
-$EndComp
-$Comp
 L L-TYPE1 L3
 U 1 1 5155168E
@@
 $EndComp
 $Comp
-L LED LED1
-U 1 1 51551A70
-P 4100 4550
-F 0 "LED1" H 4000 4670 40  0000 L CNN
-F 1 "LED" H 4100 4470 40  0000 C CNN
-F 2 "~" H 4100 4550 60  0000 C CNN
-F 3 "~" H 4100 4550 60  0000 C CNN
-	1    4100 4550
-	0    -1   -1   0
-$EndComp
-$Comp
-L R-TYPE1 R2
-U 1 1 51551C4A
-P 5050 4600
-F 0 "R2" H 4950 4660 40  0000 L CNN
-F 1 "R-TYPE1" H 5050 4530 40  0000 C CNN
-F 2 "~" V 4980 4600 30  0000 C CNN
-F 3 "~" H 5050 4600 30  0000 C CNN
-F 4 "4.7k" H 5050 4580 35  0000 C BNN "Resistance"
-	1    5050 4600
-	1    0    0    -1
-$EndComp
-$Comp
 L L-TYPE2 L2
 U 1 1 51553EBA
@@
 $EndComp
 $Comp
-L CON-MALE-SINGLE-001 CN3
-U 1 1 5155DBCE
-P 6600 4850
-F 0 "CN3" H 6550 4930 40  0000 L CNN
-F 1 "CON-MALE-SINGLE-001" H 6650 4760 40  0000 C CNN
-F 2 "~" H 6550 4850 60  0000 C CNN
-F 3 "~" H 6550 4850 60  0000 C CNN
-	1    6600 4850
-	1    0    0    -1
-$EndComp
-$Comp
-L CON-MALE-SINGLE-002 CN2
-U 1 1 5155DBDD
-P 6600 4550
-F 0 "CN2" H 6550 4680 40  0000 L CNN
-F 1 "CON-MALE-SINGLE-002" H 6650 4410 40  0000 C CNN
-F 2 "~" H 6550 4600 60  0000 C CNN
-F 3 "~" H 6550 4600 60  0000 C CNN
-	1    6600 4550
-	1    0    0    -1
-$EndComp
-$Comp
-L CON-MALE-SINGLE-003 CN1
-U 1 1 5155DBEC
-P 6600 4150
-F 0 "CN1" H 6550 4330 40  0000 L CNN
-F 1 "CON-MALE-SINGLE-003" H 6650 3960 40  0000 C CNN
-F 2 "~" H 6550 4250 60  0000 C CNN
-F 3 "~" H 6550 4250 60  0000 C CNN
-	1    6600 4150
-	1    0    0    -1
-$EndComp
-$Comp
-L CON-FEMALE-SINGLE-001 CN7
-U 1 1 5155DBFB
-P 7450 4850
-F 0 "CN7" H 7400 4930 40  0000 L CNN
-F 1 "CON-FEMALE-SINGLE-001" H 7500 4760 40  0000 C CNN
-F 2 "~" H 7400 4850 60  0000 C CNN
-F 3 "~" H 7400 4850 60  0000 C CNN
-	1    7450 4850
-	1    0    0    -1
-$EndComp
-$Comp
-L CON-FEMALE-SINGLE-002 CN6
-U 1 1 5155DC14
-P 7450 4550
-F 0 "CN6" H 7400 4680 40  0000 L CNN
-F 1 "CON-FEMALE-SINGLE-002" H 7500 4410 40  0000 C CNN
-F 2 "~" H 7400 4600 60  0000 C CNN
-F 3 "~" H 7400 4600 60  0000 C CNN
-	1    7450 4550
-	1    0    0    -1
-$EndComp
-$Comp
-L CON-FEMALE-SINGLE-003 CN5
-U 1 1 5155DC23
-P 7450 4150
-F 0 "CN5" H 7400 4330 40  0000 L CNN
-F 1 "CON-FEMALE-SINGLE-003" H 7500 3960 40  0000 C CNN
-F 2 "~" H 7400 4250 60  0000 C CNN
-F 3 "~" H 7400 4250 60  0000 C CNN
-	1    7450 4150
-	1    0    0    -1
-$EndComp
-$Comp
-L CON-FEMALE-DOUBLE-008 CN8
-U 1 1 5155EEE5
-P 7550 5250
-F 0 "CN8" H 7400 5480 40  0000 L CNN
-F 1 "CON-FEMALE-DOUBLE-008" H 7550 5010 40  0000 C CNN
-F 2 "~" H 7500 5425 60  0000 C CNN
-F 3 "~" H 7500 5425 60  0000 C CNN
-	1    7550 5250
-	1    0    0    -1
-$EndComp
-$Comp
-L CON-MALE-DOUBLE-006 CN4
-U 1 1 5155EEF4
-P 6700 5200
-F 0 "CN4" H 6550 5380 40  0000 L CNN
-F 1 "CON-MALE-DOUBLE-006" H 6700 5010 40  0000 C CNN
-F 2 "~" H 6650 5325 60  0000 C CNN
-F 3 "~" H 6650 5325 60  0000 C CNN
-	1    6700 5200
-	1    0    0    -1
-$EndComp
-$Comp
 L +11.1V #PWR?
 U 1 1 5157A02F
@@
 	1    0    0    -1
 $EndComp
+$Comp
+L LED(PHI5) LED?
+U 1 1 51661A48
+P 4050 4550
+F 0 "LED?" H 3950 4670 40  0000 L CNN
+F 1 "LED(PHI5)" H 4050 4470 40  0000 C CNN
+F 2 "~" H 4050 4550 60  0000 C CNN
+F 3 "~" H 4050 4550 60  0000 C CNN
+	1    4050 4550
+	0    -1   -1   0
+$EndComp
+$Comp
+L C(CERA) C?
+U 1 1 51661D91
+P 4950 4850
+F 0 "C?" H 5000 4920 45  0000 L CNN
+F 1 "C(CERA)" H 5000 4775 45  0000 L CNN
+F 2 "~" H 4988 4700 30  0000 C CNN
+F 3 "~" H 4950 4850 60  0000 C CNN
+	1    4950 4850
+	1    0    0    -1
+$EndComp
+$Comp
+L C(POLE) C?
+U 1 1 5166204C
+P 4500 4850
+F 0 "C?" H 4550 4920 45  0000 L CNN
+F 1 "C(POLE)" H 4550 4775 45  0000 L CNN
+F 2 "~" H 4538 4700 30  0000 C CNN
+F 3 "~" H 4500 4850 60  0000 C CNN
+	1    4500 4850
+	1    0    0    -1
+$EndComp
+$Comp
+L C(NPOLE) C?
+U 1 1 5166205B
+P 4200 5000
+F 0 "C?" H 4250 5070 45  0000 L CNN
+F 1 "C(NPOLE)" H 4250 4925 45  0000 L CNN
+F 2 "~" H 4238 4850 30  0000 C CNN
+F 3 "~" H 4200 5000 60  0000 C CNN
+	1    4200 5000
+	1    0    0    -1
+$EndComp
+$Comp
+L R(1005M) R?
+U 1 1 5166230D
+P 5100 4350
+F 0 "R?" H 4975 4410 45  0000 L CNN
+F 1 "R(1005M)" H 5100 4280 45  0000 C CNN
+F 2 "~" V 5030 4350 30  0000 C CNN
+F 3 "~" H 5100 4350 30  0000 C CNN
+	1    5100 4350
+	1    0    0    -1
+$EndComp
+$Comp
+L CON-FEMALE-DOUBLE-10 CN?
+U 1 1 51662D14
+P 6950 4000
+F 0 "CN?" H 6800 4280 40  0000 L CNN
+F 1 "CON-FEMALE-DOUBLE-10" H 6950 3710 40  0000 C CNN
+F 2 "~" H 6900 4225 60  0000 C CNN
+F 3 "~" H 6900 4225 60  0000 C CNN
+	1    6950 4000
+	1    0    0    -1
+$EndComp
+$Comp
+L CON-MALE-DOUBLE-10 CN?
+U 1 1 51662D23
+P 6950 4700
+F 0 "CN?" H 6800 4980 40  0000 L CNN
+F 1 "CON-MALE-DOUBLE-10" H 6950 4410 40  0000 C CNN
+F 2 "~" H 6900 4925 60  0000 C CNN
+F 3 "~" H 6900 4925 60  0000 C CNN
+	1    6950 4700
+	1    0    0    -1
+$EndComp
